File: pcb/pcb.kicad_pcb (KiCad board)
At the start: 2 copper layers, 56.5 x 44.4 mm, 31 parts, among them J1 Switch 1, J10 Valves Pico, J11 12V in, J2 Power in, J3 Switches Pico, J4 Valves, J5 Switch 2, J6 Power out, J7 5V out, J8 Switch 3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

Commit message: finished board
Parts:
- added G***: LOGO, LOGO, B.Cu at (107.4, 71.9)
- J1: value Switch 1 -> S1
- J5: value Switch 2 -> S2
- J8: value Switch 3 -> S3
- J9: value Switch 4 -> S4
- moved D4 12.0 mm to (137.2, 48.3), turned to -90 degrees
Routing:
- net /M4: track 39.4 -> 46.0 mm
- net +12V: track 172.9 -> 174.6 mm
Other:
- board text added: "12V"
- board text added: "5V"
- board text added: "GND"
- board text added: "J2, J6 POWER IN & OUT (12V, 5V) J7 (OPTIONAL) POWER TO MCU J4 VALVES J10 VALVE CONTROL FROM MCU J3 SWITCH SIGNAL TO MCU J1, J5, J8, J9 SWITCHES U1 (OPTIONAL) DC/DC-REGULATOR 5V USE IF BOARD POWERED BY 12V U2 (OPTIONAL) DC/DC-REGULATOR 12V USE IF BOARD POWERED BY 5V"
- board text added: "S1"
- board text added: "S4"
- board text added: "V1"
- board text added: "V4"

Commit message: finalized pcb design
Parts:
- moved C1 7.68 mm to (121.9, 68.6)
- moved C2 7.68 mm to (121.9, 76.2)
Changed lines of the file:
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@@
 			(plot_on_all_layers_selection 0x00000000_00000000_00000000_00000000)
 			(disableapertmacros no)
-			(usegerberextensions no)
-			(usegerberattributes yes)
-			(usegerberadvancedattributes yes)
-			(creategerberjobfile yes)
+			(usegerberextensions yes)
+			(usegerberattributes no)
+			(usegerberadvancedattributes no)
+			(creategerberjobfile no)
 			(dashed_line_dash_ratio 12.000000)
 			(dashed_line_gap_ratio 3.000000)
@@
 			(sketchdnponfab yes)
 			(crossoutdnponfab yes)
-			(subtractmaskfromsilk no)
+			(subtractmaskfromsilk yes)
 			(outputformat 1)
 			(mirror no)
-			(drillshape 1)
+			(drillshape 0)
 			(scaleselection 1)
-			(outputdirectory "")
+			(outputdirectory "gerber/")
 		)
 	)
@@
 		(tags "TO-220-3 Vertical RM 2.54mm")
 		(property "Reference" "U1"
-			(at 8.89 -2.345 90)
+			(at 2.54 -4.25 90)
 			(layer "F.SilkS")
 			(effects
@@
 		)
 		(property "Value" "LMO78_05-0.5"
-			(at 2.54 -4.25 90)
+			(at 2.54 2.1 90)
 			(layer "F.SilkS")
 			(effects
@@
 	(footprint "Capacitor_SMD:C_1206_3216Metric_Pad1.33x1.80mm_HandSolder"
 		(layer "F.Cu")
-		(at 114.3 67.6025 90)
+		(at 121.92 68.58 90)
 		(descr "Capacitor SMD 1206 (3216 Metric), square (rectangular) end terminal, IPC_7351 nominal with elongated pad for handsoldering. (Body size source: IPC-SM-782 page 76, https://www.pcb-3d.com/wordpress/wp-content/uploads/ipc-sm-782a_amendment_1_and_2.pdf), generated with kicad-footprint-generator")
 		(tags "capacitor handsolder")
 		(property "Reference" "C1"
-			(at -2.2475 -1.905 90)
+			(at -2.2475 1.905 90)
 			(layer "F.SilkS")
 			(effects
@@
 		)
 		(property "Value" "10u"
-			(at 0.9275 -1.905 90)
+			(at 0.9275 1.905 90)
 			(layer "F.SilkS")
 			(effects
@@
 	(footprint "Capacitor_SMD:C_1206_3216Metric_Pad1.33x1.80mm_HandSolder"
 		(layer "F.Cu")
-		(at 114.3 77.1775 -90)
+		(at 121.92 76.2 -90)
 		(descr "Capacitor SMD 1206 (3216 Metric), square (rectangular) end terminal, IPC_7351 nominal with elongated pad for handsoldering. (Body size source: IPC-SM-782 page 76, https://www.pcb-3d.com/wordpress/wp-content/uploads/ipc-sm-782a_amendment_1_and_2.pdf), generated with kicad-footprint-generator")
 		(tags "capacitor handsolder")
 		(property "Reference" "C2"
-			(at 2.8325 1.905 90)
+			(at 2.8325 -1.905 90)
 			(layer "F.SilkS")
 			(effects
@@
 		)
 		(property "Value" "22u"
-			(at -0.9775 1.85 90)
+			(at -0.9775 -1.905 90)
 			(layer "F.SilkS")
 			(effects
@@
 	)
 	(gr_text "J2, J6 POWER IN & OUT (12V, 5V)\nJ7 (OPTIONAL) POWER TO MCU\nJ4 VALVES\nJ10 VALVE CONTROL FROM MCU\nJ3 SWITCH SIGNAL TO MCU\nJ1, J5, J8, J9 SWITCHES\n\nU1 (OPTIONAL) DC/DC-REGULATOR 5V\n    USE IF BOARD POWERED BY 12V\nU2 (OPTIONAL) DC/DC-REGULATOR 12V\n    USE IF BOARD POWERED BY 5V"
-		(at 144.272 48.006 0)
-		(layer "B.SilkS")
+		(at 146.05 46.99 0)
+		(layer "User.1")
 		(effects
 			(font
@@
 				(thickness 0.15)
 			)
-			(justify left mirror)
+			(justify left)
 		)
 	)
@@
 	)
 	(segment
-		(start 116.35 69.165)
-		(end 117.035 69.85)
-		(width 0.4064)
-		(layer "F.Cu")
-		(net 1)
-	)
-	(segment
 		(start 97.79 40.1212)
 		(end 97.79 41.91)
@@
 	)
 	(segment
-		(start 103.54 68.58)
-		(end 113.715 68.58)
-		(width 0.4064)
-		(layer "F.Cu")
-		(net 1)
-	)
-	(segment
 		(start 128.465 69.85)
 		(end 138.755 69.85)
@@
 	)
 	(segment
-		(start 113.715 68.58)
-		(end 114.3 69.165)
-		(width 0.4064)
-		(layer "F.Cu")
-		(net 1)
-	)
-	(segment
 		(start 106.0012 40.1212)
 		(end 102.79 40.1212)
@@
 	)
 	(segment
-		(start 114.3 69.165)
-		(end 116.35 69.165)
+		(start 103.54 68.58)
+		(end 115.765 68.58)
 		(width 0.4064)
 		(layer "F.Cu")
@@
 	)
 	(segment
+		(start 115.765 68.58)
+		(end 117.035 69.85)
+		(width 0.4064)
+		(layer "F.Cu")
+		(net 1)
+	)
+	(segment
 		(start 115.062 42.672)
 		(end 131.572 42.672)
@@
 	)
 	(segment
-		(start 92.71 76.2)
-		(end 113.715 76.2)
-		(width 0.4064)
-		(layer "F.Cu")
-		(net 3)
-	)
-	(segment
-		(start 114.985 74.93)
-		(end 114.3 75.615)
-		(width 0.4064)
-		(layer "F.Cu")
-		(net 3)
-	)
-	(segment
 		(start 141.659169 38.9762)
 		(end 144.1608 41.477831)
@@
 	)
 	(segment
-		(start 113.715 76.2)
-		(end 114.3 75.615)
+		(start 117.035 74.93)
+		(end 115.765 76.2)
 		(width 0.4064)
 		(layer "F.Cu")
@@
 	)
 	(segment
-		(start 117.035 74.93)
-		(end 114.985 74.93)
+		(start 115.765 76.2)
+		(end 92.71 76.2)
 		(width 0.4064)
 		(layer "F.Cu")
